Commit message: rebuild

File: src/robot_description/urdf/robot.urdf.xacro (robot description, xacro)
@@ -1,57 +1,51 @@
 <?xml version="1.0"?>
-<robot xmlns:xacro="http://www.ros.org/wiki/xacro" name="diffbot">
-  <!-- ========================
-       Top-level robot description.
-       This file is simulator-agnostic except for the optional
-       Gazebo plugins which are injected only when use_sim=true.
-       ======================== -->
+<robot xmlns:xacro="http://www.ros.org/wiki/xacro" name="gobot">
   <xacro:arg name="use_sim" default="true"/>
-  <xacro:arg name="use_lidar" default="true"/>
-  <xacro:arg name="use_camera" default="true"/>
-  <xacro:property name="use_sim_enabled" value="$(arg use_sim)"/>
-  <xacro:property name="use_lidar_enabled" value="$(arg use_lidar)"/>
-  <xacro:property name="use_camera_enabled" value="$(arg use_camera)"/>
   <xacro:property name="wheel_radius" value="0.08"/>
-  <xacro:property name="wheel_width" value="0.04"/>
-  <xacro:property name="wheel_separation" value="0.30"/>
-  <xacro:property name="chassis_length" value="0.35"/>
-  <xacro:property name="chassis_width" value="0.25"/>
-  <xacro:property name="chassis_height" value="0.10"/>
-  <xacro:property name="chassis_mass" value="2.0"/>
-  <xacro:property name="wheel_mass" value="0.3"/>
-  <xacro:property name="caster_mass" value="0.1"/>
-  <!-- Include modular xacros -->
-  <xacro:include filename="$(find robot_description)/urdf/chassis.xacro"/>
-  <xacro:include filename="$(find robot_description)/urdf/gazebo/materials.xacro"/>
-  <xacro:include filename="$(find robot_description)/urdf/gazebo/plugins.xacro"/>
-  <xacro:include filename="$(find robot_description)/urdf/sensors/lidar.xacro"/>
-  <xacro:include filename="$(find robot_description)/urdf/sensors/camera.xacro"/>
-  <!-- Base footprint -->
+  <material name="blue"><color rgba="0.05 0.25 0.8 1"/></material>
+  <material name="black"><color rgba="0.02 0.02 0.02 1"/></material>
+  <material name="grey"><color rgba="0.5 0.5 0.5 1"/></material>
+  <material name="red"><color rgba="0.8 0.05 0.05 1"/></material>
   <link name="base_footprint"/>
-  <!-- Chassis and wheels -->
-  <xacro:chassis
-    wheel_radius="${wheel_radius}"
-    wheel_width="${wheel_width}"
-    wheel_separation="${wheel_separation}"
-    chassis_length="${chassis_length}"
-    chassis_width="${chassis_width}"
-    chassis_height="${chassis_height}"
-    chassis_mass="${chassis_mass}"
-    wheel_mass="${wheel_mass}"
-    caster_mass="${caster_mass}"/>
-  <!-- Sensors -->
-  <xacro:if value="${use_lidar_enabled}">
-    <xacro:lidar parent="base_link" x="0.12" y="0" z="0.12" radius="0.04"/>
-  </xacro:if>
-  <xacro:if value="${use_camera_enabled}">
-    <xacro:camera parent="base_link" x="0.10" y="0" z="0.08"/>
-  </xacro:if>
-  <!-- Gazebo-specific plugins (only when running in simulation) -->
-  <xacro:if value="${use_sim_enabled}">
-    <xacro:gazebo_plugins
-      wheel_radius="${wheel_radius}"
-      wheel_separation="${wheel_separation}"
-      left_joint="left_wheel_joint"
-      right_joint="right_wheel_joint"/>
-  </xacro:if>
+  <link name="base_link">
+    <visual><origin xyz="0 0 0.08"/><geometry><box size="0.35 0.25 0.16"/></geometry><material name="blue"/></visual>
+    <collision><origin xyz="0 0 0.08"/><geometry><box size="0.35 0.25 0.16"/></geometry></collision>
+    <inertial><origin xyz="0 0 0.08"/><mass value="2.0"/><inertia ixx="0.0111" ixy="0" ixz="0" iyy="0.0211" iyz="0" izz="0.0167"/></inertial>
+  </link>
+  <joint name="base_joint" type="fixed"><parent link="base_footprint"/><child link="base_link"/><origin xyz="0 0 ${wheel_radius}"/></joint>
+  <link name="left_wheel"><visual><origin rpy="1.5708 0 0"/><geometry><cylinder radius="${wheel_radius}" length="0.04"/></geometry><material name="black"/></visual><collision><origin rpy="1.5708 0 0"/><geometry><cylinder radius="${wheel_radius}" length="0.04"/></geometry></collision><inertial><mass value="0.3"/><inertia ixx="0.0006" ixy="0" ixz="0" iyy="0.0006" iyz="0" izz="0.00096"/></inertial></link>
+  <joint name="left_wheel_joint" type="continuous"><parent link="base_link"/><child link="left_wheel"/><origin xyz="0 0.15 0"/><axis xyz="0 1 0"/><dynamics damping="0.1" friction="0.02"/></joint>
+  <link name="right_wheel"><visual><origin rpy="1.5708 0 0"/><geometry><cylinder radius="${wheel_radius}" length="0.04"/></geometry><material name="black"/></visual><collision><origin rpy="1.5708 0 0"/><geometry><cylinder radius="${wheel_radius}" length="0.04"/></geometry></collision><inertial><mass value="0.3"/><inertia ixx="0.0006" ixy="0" ixz="0" iyy="0.0006" iyz="0" izz="0.00096"/></inertial></link>
+  <joint name="right_wheel_joint" type="continuous"><parent link="base_link"/><child link="right_wheel"/><origin xyz="0 -0.15 0"/><axis xyz="0 1 0"/><dynamics damping="0.1" friction="0.02"/></joint>
+  <link name="caster_wheel"><visual><geometry><sphere radius="0.045"/></geometry><material name="grey"/></visual><collision><geometry><sphere radius="0.045"/></geometry></collision><inertial><mass value="0.1"/><inertia ixx="0.00008" ixy="0" ixz="0" iyy="0.00008" iyz="0" izz="0.00008"/></inertial></link>
+  <joint name="caster_joint" type="fixed"><parent link="base_link"/><child link="caster_wheel"/><origin xyz="-0.12 0 -0.032"/></joint>
+  <link name="lidar_link"><visual><geometry><cylinder radius="0.04" length="0.05"/></geometry><material name="red"/></visual><collision><geometry><cylinder radius="0.04" length="0.05"/></geometry></collision><inertial><mass value="0.05"/><inertia ixx="0.00003" ixy="0" ixz="0" iyy="0.00003" iyz="0" izz="0.00004"/></inertial></link>
+  <joint name="lidar_joint" type="fixed"><parent link="base_link"/><child link="lidar_link"/><origin xyz="0.10 0 0.20"/></joint>
+  <link name="camera_link"><visual><geometry><box size="0.05 0.08 0.04"/></geometry><material name="black"/></visual><inertial><mass value="0.05"/><inertia ixx="0.00001" ixy="0" ixz="0" iyy="0.00001" iyz="0" izz="0.00001"/></inertial></link>
+  <joint name="camera_joint" type="fixed"><parent link="base_link"/><child link="camera_link"/><origin xyz="0.12 0 0.18"/></joint>
+  <link name="camera_optical_frame"/><joint name="camera_optical_joint" type="fixed"><parent link="camera_link"/><child link="camera_optical_frame"/><origin rpy="-1.5708 0 -1.5708"/></joint>
+  <gazebo reference="left_wheel"><mu1>0.9</mu1><mu2>0.9</mu2></gazebo>
+  <gazebo reference="right_wheel"><mu1>0.9</mu1><mu2>0.9</mu2></gazebo>
+  <gazebo>
+    <plugin name="diff_drive" filename="libgazebo_ros_diff_drive.so">
+      <ros><remapping>cmd_vel:=/cmd_vel</remapping><remapping>odom:=/odom</remapping></ros>
+      <update_rate>50</update_rate><left_joint>left_wheel_joint</left_joint><right_joint>right_wheel_joint</right_joint>
+      <wheel_separation>0.30</wheel_separation><wheel_diameter>0.16</wheel_diameter>
+      <max_wheel_torque>5.0</max_wheel_torque><max_wheel_acceleration>2.0</max_wheel_acceleration>
+      <publish_odom>true</publish_odom><publish_odom_tf>true</publish_odom_tf><publish_wheel_tf>true</publish_wheel_tf>
+      <odometry_frame>odom</odometry_frame><robot_base_frame>base_footprint</robot_base_frame>
+    </plugin>
+  </gazebo>
+  <gazebo reference="lidar_link">
+    <sensor name="lidar" type="ray"><always_on>true</always_on><update_rate>10</update_rate><visualize>false</visualize>
+      <ray><scan><horizontal><samples>360</samples><resolution>1</resolution><min_angle>-3.14159</min_angle><max_angle>3.14159</max_angle></horizontal></scan><range><min>0.12</min><max>10.0</max><resolution>0.01</resolution></range></ray>
+      <plugin name="lidar_controller" filename="libgazebo_ros_ray_sensor.so"><ros><remapping>~/out:=/scan</remapping></ros><output_type>sensor_msgs/LaserScan</output_type><frame_name>lidar_link</frame_name></plugin>
+    </sensor>
+  </gazebo>
+  <gazebo reference="camera_link">
+    <sensor name="camera" type="camera"><always_on>true</always_on><update_rate>15</update_rate><visualize>false</visualize>
+      <camera><horizontal_fov>1.047</horizontal_fov><image><width>640</width><height>480</height><format>R8G8B8</format></image><clip><near>0.05</near><far>20.0</far></clip></camera>
+      <plugin name="camera_controller" filename="libgazebo_ros_camera.so"><ros><remapping>image_raw:=/camera/image</remapping><remapping>camera_info:=/camera/camera_info</remapping></ros><camera_name>camera</camera_name><frame_name>camera_optical_frame</frame_name></plugin>
+    </sensor>
+  </gazebo>
 </robot>
